File: Rocket/Boards/Onboard_Radio/_restore_backup_2026-05-20T13-01-22-586/can_termination.kicad_sch (KiCad schematic)
At the start: 16 parts, among them J10 M80-5301042, J7 CAN1_T, J8 CAN2_T, J9 M80-5301042, U1 TCAN1046

Commit message: schematic bom needs updating and traces need finishing
Parts:
- removed F2: 5A, Fuse:Fuse_1206_3216Metric, symbol Device:Fuse
- removed J10, J9: M80-5301042, Connector_Harwin:Harwin_LTek-Male_2x05_P2.00mm_Vertical, symbol Connector_Generic:Conn_01x10
- added F1: 5A, Fuse:Fuse_1206_3216Metric, symbol Device:Fuse
- added J3, J6: DB9 Microfit, Connector_Dsub:DSUB-9_Pins_Horizontal_P2.77x2.84mm_EdgePinOffset7.70mm_Housed_MountingHolesOffset9.12mm, symbol Connector:DE9_Socket
- renumbered C19 to C100, C20 to C101, J7 to J1, J8 to J2, R1 to R100, R5 to R101, R6 to R102, R2 to R103, R7 to R104, R8 to R105, U1 to U2
Connections:
- net CAN1_AUX: now also J6.3
- net CAN2_AUX: now also J3.3
- net CANH1: now also J3.6, J6.6
- net CANH2: now also J3.8, J6.8
- net CANL1: now also J3.7, J6.7
- net CANL2: now also J3.9, J6.9
- net CAN_PWR_IN: now also F1.1
- net GND: now also J3.2, J3.4, J6.2, J6.4
- new net: F1.2, J3.1, J3.5, J6.1, J6.5
- no-connect marks 4 -> 2
