File: Rocket/Boards/Onboard_Radio/_restore_backup_2026-05-20T13-01-22-586/mircocontroller.kicad_sch (KiCad schematic)
At the start: 32 parts, among them J3 USB_B_Micro, J4 SWD JST PH, U4 STM32H562RGT6, Y2 12MHz

Commit message: schematic bom needs updating and traces need finishing
Parts:
- renumbered C21 to C106, C22 to C107, C23 to C109, C25 to C110, C24 to C111, C26 to C112, C27 to C113, C28 to C114, C29 to C115, C30 to C116, C31 to C121, C32 to C122, C33 to C124, C34 to C125, J3 to J4, J4 to J5, R9 to R108, R12 to R120, R14 to R126, R15 to R127, R16 to R128, R13 to R129, R10 to R130, R11 to R140, TP1 to TP5, TP2 to TP6, U4 to U8, Y2 to Y123
Connections:
- net Antenna Switch: no longer U8.35 (PB14)
- net LED1: now also U8.9 (PC1); no longer U8.15 (PA1)
- net LED2: now also U8.10 (PC2); no longer U8.16 (PA2)
- no-connect marks 33 -> 3
Other:
- note removed: "WTF IS THIS GOING TO GND????"
- note removed: "check these are gpio"
- note removed: "make these diff pairs in pcb"
