File: Rocket/Boards/Onboard_Radio/_restore_backup_2026-05-20T13-02-04-446/can_termination.kicad_sch (KiCad schematic)
At the start: 16 parts, among them J10 M80-5301042, J7 CAN1_T, J8 CAN2_T, J9 M80-5301042, U1 TCAN1046

Commit message: schematic bom needs updating and traces need finishing
Parts:
- removed F2: 5A, Fuse:Fuse_1206_3216Metric, symbol Device:Fuse
- removed J10, J9: M80-5301042, Connector_Harwin:Harwin_LTek-Male_2x05_P2.00mm_Vertical, symbol Connector_Generic:Conn_01x10
- added F1: 5A, Fuse:Fuse_1206_3216Metric, symbol Device:Fuse
- added J1, J2: DB9 Microfit, Connector_Dsub:DSUB-9_Pins_Horizontal_P2.77x2.84mm_EdgePinOffset7.70mm_Housed_MountingHolesOffset9.12mm, symbol Connector:DE9_Socket
- renumbered J7 to J1, J8 to J2
Connections:
- net CAN1_AUX: now also J2.3
- net CAN2_AUX: now also J1.3
- net CANH1: now also J1.6, J2.6
- net CANH2: now also J1.8, J2.8
- net CANL1: now also J1.7, J2.7
- net CANL2: now also J1.9, J2.9
- net CAN_PWR_IN: now also F1.1
- net GND: now also J1.2, J1.4, J2.2, J2.4
- new net: F1.2, J1.1, J1.5, J2.1, J2.5
- no-connect marks 4 -> 2
