File: Rocket/Boards/Onboard_Radio/_restore_backup_2026-05-20T13-02-04-446/power_connection.kicad_sch (KiCad schematic)
At the start: 1 part, among them J5 Conn_01x08

Commit message: schematic bom needs updating and traces need finishing
Parts:
- J5: footprint Connector_PinSocket_2.54mm:PinSocket_1x08_P2.54mm_Vertical -> (none)
Changed lines of the file:
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@@
 			)
 		)
-		(property "Footprint" "Connector_PinSocket_2.54mm:PinSocket_1x08_P2.54mm_Vertical"
+		(property "Footprint" ""
 			(at 125.73 96.52 0)
 			(hide yes)
