File: Rocket/Boards/Onboard_Radio/mircocontroller.kicad_sch (KiCad schematic)
At the start: 32 parts, among them J3 USB_B_Micro, J4 SWD JST PH, U4 STM32H562RGT6, Y2 12MHz

Commit message: pcb done, need schematic review
Parts:
- removed TP1: BOOT0, symbol Connector:TestPoint_Small
- C33, C34, R12: footprint (none) -> Resistor_SMD:R_0603_1608Metric
- TP2: footprint TestPoint:TestPoint_Pad_1.5x1.5mm -> TestPoint:TestPoint_Pad_1.0x1.0mm
