File: Rocket/Boards/Onboard_Radio/can_termination.kicad_sch (KiCad schematic)
At the start: 16 parts, among them J10 M80-5301042, J7 CAN1_T, J8 CAN2_T, J9 M80-5301042, U1 TCAN1046

Commit message: can bus updeated
Parts:
- added C35, C36: 100nF, Capacitor_SMD:C_0603_1608Metric, symbol Device:C
- added F3: 5A, Fuse:Fuse_1206_3216Metric, symbol Device:Fuse
- added J11: CAN1_T, Connector_PinHeader_2.54mm:PinHeader_1x02_P2.54mm_Vertical, symbol Connector_Generic:Conn_01x02
- added J12: CAN2_T, Connector_PinHeader_2.54mm:PinHeader_1x02_P2.54mm_Vertical, symbol Connector_Generic:Conn_01x02
- added J13, J14: M80-5301042, Connector_Harwin:Harwin_LTek-Male_2x05_P2.00mm_Vertical, symbol Connector_Generic:Conn_01x10
- added R22, R23: 120R, Resistor_SMD:R_0603_1608Metric, symbol Device:R
- added U5: TCAN1046, Library:Texas_DYY0014A_TSOT-23-14, symbol Interface_CAN_LIN:TCAN1046AV-Q1
Connections:
- net +3V3: now also R5.1, R6.1, C36.1, U5.14 (STB1), U5.3 (VCC), U5.8 (STB2)
- net +5V: now also C35.1, U5.11 (VIO)
- net CAN1_AUX: now also J13.3 (Pin_3)
- net CAN1_RX: now also U5.4 (RXD1)
- net CAN1_TX: now also U5.1 (TXD1)
- net CAN2_AUX: now also J14.3 (Pin_3)
- net CAN_PWR_IN: now also F3.1
- net GND: now also C35.2, C36.2, J13.2 (Pin_2), J13.4 (Pin_4), J14.2 (Pin_2), J14.4 (Pin_4), U5.2 (GND), U5.5 (GND)
- net CAN2_TX: now reaches U1.6 (TXD2)
- net CAN2_TX: now also U5.6 (TXD2); no longer R5.1
- net CAN2_RX: now reaches U1.7 (RXD2)
- net CAN2_RX: now also U5.7 (RXD2); no longer R6.1
- net CANH1 renamed CAN1H
- net CAN1H: now also J11.1 (Pin_1), J13.6 (Pin_6), J14.6 (Pin_6), U5.13 (CANH1)
- net CANH2 renamed CAN2H
- net CAN2H: now also J13.8 (Pin_8), J14.8 (Pin_8), R23.1, U5.10 (CANH2)
- net CANL1 renamed CAN1L
- net CAN1L: now also J13.7 (Pin_7), J14.7 (Pin_7), R22.2, U5.12 (CANL1)
- net CANL2 renamed CAN2L
- net CAN2L: now also J12.1 (Pin_1), J13.9 (Pin_9), J14.9 (Pin_9), U5.9 (CANL2)
- new net: F3.2, J13.1 (Pin_1), J13.5 (Pin_5), J14.1 (Pin_1), J14.5 (Pin_5)
- new net: J12.2 (Pin_2), R23.2
- new net: J11.2 (Pin_2), R22.1
- no-connect marks 4 -> 6
Other:
- title: (none) -> CAN Transceiver
- moved on the sheet: C19, C20, F2, J10, J7, J8, J9, JP1, JP2, R1, R2, R7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

Commit message: pcb updates
Parts:
- removed C35, C36: 100nF, Capacitor_SMD:C_0603_1608Metric, symbol Device:C
- removed F3: 5A, Fuse:Fuse_1206_3216Metric, symbol Device:Fuse
- removed J11: CAN1_T, Connector_PinHeader_2.54mm:PinHeader_1x02_P2.54mm_Vertical, symbol Connector_Generic:Conn_01x02
- removed J12: CAN2_T, Connector_PinHeader_2.54mm:PinHeader_1x02_P2.54mm_Vertical, symbol Connector_Generic:Conn_01x02
- removed J13, J14: M80-5301042, Connector_Harwin:Harwin_LTek-Male_2x05_P2.00mm_Vertical, symbol Connector_Generic:Conn_01x10
- removed R22, R23: 120R, Resistor_SMD:R_0603_1608Metric, symbol Device:R
- removed R5, R6: 100K, Resistor_SMD:R_0603_1608Metric, symbol Device:R
- removed U5: TCAN1046, Library:Texas_DYY0014A_TSOT-23-14, symbol Interface_CAN_LIN:TCAN1046AV-Q1
Connections:
- net CAN1H renamed CANH1
- net CAN1L renamed CANL1
- net CAN2H renamed CANH2
- net CAN2L renamed CANL2
- no-connect marks 6 -> 4

Commit message: schematic ready for review
Parts:
- removed R2: 100K, Resistor_SMD:R_0603_1608Metric, symbol Device:R
- J10, J9: value M80-5301042 -> M80; MPN (none) -> M80-5301042; Manufacturer (none) -> Harwin Inc.
Connections:
- net +3V3: no longer R1.1
- net CAN2_RX: no longer names the net of U1.7 (RXD2)
- net CAN2_TX: no longer names the net of U1.6 (TXD2)
- new net CAN_STB1: R1.1
- no-connect marks 4 -> 7

Commit message: everything minus trace impedance and via stictching
Parts:
- removed J7: CAN1_T, Connector_PinHeader_2.54mm:PinHeader_1x02_P2.54mm_Vertical, symbol Connector_Generic:Conn_01x02
- removed J8: CAN2_T, Connector_PinHeader_2.54mm:PinHeader_1x02_P2.54mm_Vertical, symbol Connector_Generic:Conn_01x02
- removed JP1, JP2: CH SEL, Jumper:SolderJumper-3_P1.3mm_Bridged12_RoundedPad1.0x1.5mm, symbol Jumper:SolderJumper_3_Bridged12
- added JP5, JP7: SolderJumper_2_Open, Jumper:SolderJumper-2_P1.3mm_Open_RoundedPad1.0x1.5mm, symbol Jumper:SolderJumper_2_Open
- added JP8, JP9: CH SEL, Jumper:SolderJumper-3_P1.3mm_Open_RoundedPad1.0x1.5mm, symbol Jumper:SolderJumper_3_Open
- J10, J9: footprint Connector_Harwin:Harwin_LTek-Male_2x05_P2.00mm_Vertical -> Library:HARWIN_M80-5011005
Connections:
- net CANH: now also JP8.2 (C)
- net CANH1: now also JP5.2 (B), JP8.1 (A)
- net CANH2: now also JP8.3 (B)
- net CANL: now also JP9.2 (C)
- net CANL1: now also JP9.1 (A)
- net CANL2: now also JP7.1 (A), JP9.3 (B)
- net at R7.1: now also JP5.1 (A)
- net at R8.2: now also JP7.2 (B)
Other:
- note removed: "Could look into picolock connectors"

Commit message: needs pcb and schematic review
Parts:
- C19, C20: LCSC Part # (none) -> C16194197
- F2: LCSC Part # (none) -> C3166463
- J10, J9: LCSC Part # (none) -> C17382082
- R1: LCSC Part # (none) -> C237792
- R7, R8: LCSC Part # (none) -> C3995226
- U1: LCSC Part # (none) -> C3233845
Changed lines of the file:
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@@
 			)
 		)
-		(property "LCSC Part #" ""
+		(property "LCSC Part #" "C16194197"
 			(at 93.98 74.93 0)
 			(hide yes)
@@
 			)
 		)
-		(property "LCSC Part #" ""
+		(property "LCSC Part #" "C237792"
 			(at 101.6 95.25 90)
 			(hide yes)
@@
 			)
 		)
-		(property "LCSC Part #" ""
+		(property "LCSC Part #" "C16194197"
 			(at 69.85 74.93 0)
 			(hide yes)
@@
 			)
 		)
-		(property "LCSC Part #" ""
+		(property "LCSC Part #" "C3233845"
 			(at 83.82 104.14 0)
 			(hide yes)
@@
 			)
 		)
+		(property "LCSC Part #" "C17382082"
+			(at 217.17 64.77 90)
+			(hide yes)
+			(show_name no)
+			(do_not_autoplace no)
+			(effects
+				(font
+					(size 1.27 1.27)
+				)
+			)
+		)
 		(pin "2"
 		)
@@
 			)
 		)
-		(property "LCSC Part #" ""
+		(property "LCSC Part #" "C3166463"
 			(at 240.03 123.19 90)
 			(hide yes)
@@
 		)
 		(property "Manufacturer" "Harwin Inc."
+			(at 217.17 135.89 90)
+			(hide yes)
+			(show_name no)
+			(do_not_autoplace no)
+			(effects
+				(font
+					(size 1.27 1.27)
+				)
+			)
+		)
+		(property "LCSC Part #" "C17382082"
 			(at 217.17 135.89 90)
 			(hide yes)
@@
 			)
 		)
-		(property "LCSC Part #" ""
+		(property "LCSC Part #" "C3995226"
 			(at 161.29 93.98 0)
 			(hide yes)
@@
 			)
 		)
-		(property "LCSC Part #" ""
+		(property "LCSC Part #" "C3995226"
 			(at 163.83 105.41 0)
 			(hide yes)
