File: Rocket/Boards/Onboard_Radio/power_connection.kicad_sch (KiCad schematic)
At the start: 1 part, among them J5 Conn_01x08

Commit message: can bus updeated
Other:
- title: (none) -> Power Input
Changed lines of the file:
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@@
 	(generator_version "10.0")
 	(paper "A4")
+	(title_block
+		(title "Power Input")
+		(date "2026-05-28")
+		(rev "A")
+	)
 	(no_connect
 		(at 143.51 99.06)

Commit message: updates
Parts:
- removed J5: Conn_01x08, Connector_PinSocket_2.54mm:PinSocket_1x08_P2.54mm_Vertical, symbol Connector_Generic:Conn_01x08
- added C35, C36, C37, C38: 1uF, Capacitor_SMD:C_0603_1608Metric, symbol Device:C
- added C39: 0.1uF, Capacitor_SMD:C_0603_1608Metric, symbol Device:C
- added C40: 0.33uF, Capacitor_SMD:C_0603_1608Metric, symbol Device:C
- added FB1: FerriteBead, symbol Device:FerriteBead
- added J11, J5: MICROFIT, Connector_Molex:Molex_Micro-Fit_3.0_43045-0412_2x02_P3.00mm_Vertical, symbol Connector_Generic:Conn_02x02_Counter_Clockwise
- added JP3, JP4, JP6: SolderJumper, Jumper:SolderJumper-3_P1.3mm_Open_Pad1.0x1.5mm, symbol Jumper:SolderJumper_3_Open
- added U5, U6: MIC5365-3.3YC5, Package_TO_SOT_SMD:SOT-353_SC-70-5, symbol Regulator_Linear:MIC5365-3.3YC5
- added U7: AS78L05RTR-E1, Package_TO_SOT_SMD:SOT-89-3, symbol Regulator_Linear:MIC5365-3.3YC5
Connections:
- net GND: now also C35.2, C36.2, C37.2, C38.2, C39.2, C40.2, J11.2 (Pin_2), J5.2 (Pin_2), J5.3 (Pin_3), U5.2 (GND), U6.2 (GND), U7.2 (GND)
- new net: C37.1, JP6.2 (C), U6.1 (VIN)
- new net: C38.1, FB1.2, U6.5 (VOUT)
- new net +3V3A_Input: FB1.1
- new net +3V3_In: J11.4 (Pin_4), JP3.1 (A)
- new net +3V3_Input: JP3.2 (C)
- new net +3V3_LDO: C35.1, JP3.3 (B), U5.5 (VOUT)
- new net +5V_In: J11.3 (Pin_3), JP4.1 (A), JP6.3 (B)
- new net +5V_Input: JP4.2 (C)
- new net +5V_LDO: C36.1, C39.1, JP4.3 (B), JP6.1 (A), U5.1 (VIN), U7.5 (VOUT)
- new net +7V4_Input: J11.1 (Pin_1)
- new net +V_In: C40.1, J5.1 (Pin_1), U7.1 (VIN)
- new net 3V3A_LDO_EN: U6.3 (EN)
- new net 3V3_LDO_EN: U5.3 (EN)
- new net 5V_LDO_EN: U7.3 (EN)
- no-connect marks 3 -> 1
Other:
- note added: "5V In, 3V3 Out"
- note added: "5V In, 3V3A Out"
- note added: "7V4 In, 5V Out"
- note added: "Battery Input"
- note added: "Connector Inputs"
- note added: "Power Input"
- note added: "Voltage Regs"
- note added: "Voltage Selection"

Commit message: everything minus trace impedance and via stictching
Parts:
- removed FB1: FerriteBead, symbol Device:FerriteBead
- JP3, JP4, JP6: footprint Jumper:SolderJumper-3_P1.3mm_Open_Pad1.0x1.5mm -> Jumper:SolderJumper-3_P1.3mm_Open_RoundedPad1.0x1.5mm
Connections:
- net 5V_LDO_EN is gone; now on net +V_In: U7.3 (VIN)
- net +3V3A_Input: now also C38.1, U6.5 (VOUT)
- net +5V_LDO: now also U7.1 (VOUT); no longer U7.5 (VOUT)
- net +V_In: no longer U7.1 (VIN)
Changed lines of the file:
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@@
+	)
+	(junction
+		(at 109.22 43.18)
+		(diameter 0)
+		(color 0 0 0 0)
+	)
+	(junction
+		(at 45.72 57.15)
+		(diameter 0)
+		(color 0 0 0 0)
+	)
+	(junction
+		(at 143.51 43.18)
+		(diameter 0)
+		(color 0 0 0 0)
+	)
+	(junction
+		(at 102.87 165.1)
+		(diameter 0)
+		(color 0 0 0 0)
+	)
+	(junction
+		(at 107.95 106.68)
+		(diameter 0)
+		(color 0 0 0 0)
+	)
+	(junction
+		(at 142.24 165.1)
+		(diameter 0)
+		(color 0 0 0 0)
 	)
 	(junction
@@
 		(color 0 0 0 0)
 	)
-	(junction
-		(at 109.22 43.18)
-		(diameter 0)
-		(color 0 0 0 0)
-	)
-	(junction
-		(at 45.72 57.15)
-		(diameter 0)
-		(color 0 0 0 0)
-	)
-	(junction
-		(at 143.51 43.18)
-		(diameter 0)
-		(color 0 0 0 0)
-	)
-	(junction
-		(at 102.87 165.1)
-		(diameter 0)
-		(color 0 0 0 0)
-	)
-	(junction
-		(at 107.95 106.68)
-		(diameter 0)
-		(color 0 0 0 0)
-	)
-	(junction
-		(at 142.24 165.1)
-		(diameter 0)
-		(color 0 0 0 0)
-	)
 	(no_connect
 		(at 52.07 50.8)
@@
 	(wire
 		(pts
+			(xy 113.03 125.73) (xy 115.57 125.73)
+		)
+		(stroke
+			(width 0)
+			(type default)
+		)
+	)
+	(wire
+		(pts
 			(xy 49.53 125.73) (xy 59.69 125.73)
 		)
@@
 	(wire
 		(pts
-			(xy 104.14 184.15) (xy 115.57 184.15)
-		)
-		(stroke
-			(width 0)
-			(type default)
-		)
-	)
-	(wire
-		(pts
 			(xy 125.73 116.84) (xy 125.73 119.38)
 		)
@@
 	(wire
 		(pts
-			(xy 139.7 106.68) (xy 148.59 106.68)
+			(xy 139.7 106.68) (xy 162.56 106.68)
 		)
 		(stroke
@@
 	(wire
 		(pts
-			(xy 101.6 125.73) (xy 115.57 125.73)
-		)
-		(stroke
-			(width 0)
-			(type default)
-		)
-	)
-	(wire
-		(pts
 			(xy 208.28 92.71) (xy 231.14 92.71)
 		)
@@
 	(wire
 		(pts
-			(xy 116.84 62.23) (xy 116.84 48.26)
+			(xy 116.84 60.96) (xy 116.84 48.26)
 		)
 		(stroke
@@
 	(wire
 		(pts
-			(xy 156.21 106.68) (xy 168.91 106.68)
-		)
-		(stroke
-			(width 0)
-			(type default)
-		)
-	)
-	(wire
-		(pts
-			(xy 115.57 170.18) (xy 115.57 184.15)
-		)
-		(stroke
-			(width 0)
-			(type default)
-		)
-	)
-	(wire
-		(pts
 			(xy 125.73 175.26) (xy 125.73 176.53)
 		)
@@
 	(wire
 		(pts
-			(xy 102.87 62.23) (xy 116.84 62.23)
+			(xy 114.3 60.96) (xy 116.84 60.96)
 		)
 		(stroke
@@
 		)
 	)
-	(label "3V3A_LDO_EN"
-		(at 101.6 125.73 0)
-		(effects
-			(font
-				(size 1.27 1.27)
-			)
-			(justify left bottom)
-		)
-	)
 	(label "+3V3A_LDO"
 		(at 208.28 83.82 0)
@@
 		)
 	)
-	(label "5V_LDO_EN"
-		(at 104.14 184.15 0)
-		(effects
-			(font
-				(size 1.27 1.27)
-			)
-			(justify left bottom)
-		)
-	)
 	(label "+5V_LDO"
 		(at 208.28 92.71 0)
@@
 	)
 	(label "+3V3A_LDO"
-		(at 168.91 106.68 180)
+		(at 162.56 106.68 180)
 		(effects
 			(font
@@
 			)
 			(justify right bottom)
-		)
-	)
-	(label "3V3_LDO_EN"
-		(at 102.87 62.23 0)
-		(effects
-			(font
-				(size 1.27 1.27)
-			)
-			(justify left bottom)
 		)
 	)
@@
 			)
 			(justify right bottom)
+		)
+	)
+	(hierarchical_label "3V3A_LDO_EN"
+		(shape input)
+		(at 113.03 125.73 180)
+		(effects
+			(font
+				(size 1.27 1.27)
+			)
+			(justify right)
 		)
 	)
@@
 		)
 	)
+	(hierarchical_label "3V3_LDO_EN"
+		(shape input)
+		(at 114.3 60.96 180)
+		(effects
+			(font
+				(size 1.27 1.27)
+			)
+			(justify right)
+		)
+	)
 	(hierarchical_label "+7V4_Input"
 		(shape input)
@@
 			)
 			(justify left)
-		)
-	)
-	(hierarchical_label "+3V3_Input"
-		(shape input)
-		(at 12.362 0.8096 180)
-		(effects
-			(font
-				(size 1.27 1.27)
-			)
-			(justify right)
 		)
 	)
@@
 	)
 	(symbol
+		(lib_name "Conn_02x02_Counter_Clockwise_1")
 		(lib_id "Connector_Generic:Conn_02x02_Counter_Clockwise")
 		(at 41.91 125.73 0)
@@
 			)
 		)
-		(property "Footprint" "Jumper:SolderJumper-3_P1.3mm_Open_Pad1.0x1.5mm"
+		(property "Footprint" "Jumper:SolderJumper-3_P1.3mm_Open_RoundedPad1.0x1.5mm"
 			(at 231.14 62.23 0)
 			(hide yes)
@@
 	)
 	(symbol
+		(lib_name "MIC5365-3.3YC5_1")
 		(lib_id "Regulator_Linear:MIC5365-3.3YC5")
 		(at 125.73 167.64 0)
@@
 			)
 		)
-		(pin "4"
-		)
 		(pin "2"
-		)
-		(pin "5"
 		)
 		(pin "3"
@@
 			)
 		)
-		(property "Footprint" "Jumper:SolderJumper-3_P1.3mm_Open_Pad1.0x1.5mm"
+		(property "Footprint" "Jumper:SolderJumper-3_P1.3mm_Open_RoundedPad1.0x1.5mm"
 			(at 231.14 99.06 0)
 			(hide yes)
@@
 				(path "/4940ffbe-f45f-4917-a247-12e2b32b6c35/abcae1e2-b29e-4289-bda9-47e90da98056"
 					(reference "JP4")
-					(unit 1)
-				)
-			)
-		)
-	)
-	(symbol
-		(lib_id "Device:FerriteBead")
-		(at 152.4 106.68 270)
-		(unit 1)
-		(body_style 1)
-		(exclude_from_sim no)
-		(in_bom yes)
-		(on_board yes)
-		(in_pos_files yes)
-		(dnp no)
-		(fields_autoplaced yes)
-		(property "Reference" "FB1"
-			(at 152.4508 99.06 90)
-			(show_name no)
-			(do_not_autoplace no)
-			(effects
-				(font
-					(size 1.27 1.27)
-				)
-			)
-		)
-		(property "Value" "FerriteBead"
-			(at 152.4508 101.6 90)
-			(show_name no)
-			(do_not_autoplace no)
-			(effects
-				(font
-					(size 1.27 1.27)
-				)
-			)
-		)
-		(property "Footprint" ""
-			(at 152.4 104.902 90)
-			(hide yes)
-			(show_name no)
-			(do_not_autoplace no)
-			(effects
-				(font
-					(size 1.27 1.27)
-				)
-			)
-		)
-		(property "Datasheet" ""
-			(at 152.4 106.68 0)
-			(hide yes)
-			(show_name no)
-			(do_not_autoplace no)
-			(effects
-				(font
-					(size 1.27 1.27)
-				)
-			)
-		)
-		(property "Description" "Ferrite bead"
-			(at 152.4 106.68 0)
-			(hide yes)
-			(show_name no)
-			(do_not_autoplace no)
-			(effects
-				(font
-					(size 1.27 1.27)
-				)
-			)
-		)
-		(pin "2"
-		)
-		(pin "1"
-		)
-		(instances
-			(project "rf_rocket_module"
-				(path "/4940ffbe-f45f-4917-a247-12e2b32b6c35/abcae1e2-b29e-4289-bda9-47e90da98056"
-					(reference "FB1")
 					(unit 1)
 				)
@@
 			)
 		)
-		(property "Footprint" "Jumper:SolderJumper-3_P1.3mm_Open_Pad1.0x1.5mm"
+		(property "Footprint" "Jumper:SolderJumper-3_P1.3mm_Open_RoundedPad1.0x1.5mm"
 			(at 97.79 106.68 0)
 			(hide yes)

Commit message: needs pcb and schematic review
Parts:
- C35, C36, C37, C38: LCSC Part # (none) -> C20041637; MPN (none) -> GCM033C71A104KE02J; Manufacturer (none) -> Murata Electronics; Max Temp (none) -> 125; Min Temp (none) -> -55; Voltage (none) -> 10V
- C39: value 0.1uF -> 100nF; LCSC Part # (none) -> C16194197; MPN (none) -> CL10E104KC8VPNC; Manufacturer (none) -> Samsung Electro-Mechanics; Max Temp (none) -> 150; Min Temp (none) -> -55; Voltage (none) -> 100V
- C40: LCSC Part # (none) -> C2178511; MPN (none) -> CGA3E3X7R1H334K080AB; Manufacturer (none) -> TDK; Max Temp (none) -> 125; Min Temp (none) -> -55; Voltage (none) -> 50v
- J11, J5: LCSC Part # (none) -> C277721
- U5, U6: LCSC Part # (none) -> C73103; MPN (none) -> MIC5365-3.3YC5-TR; Manufacturer (none) -> MICROCHIP
- U7: LCSC Part # (none) -> C90471; MPN (none) -> AS78L05RTR-E1; Manufacturer (none) -> DIODES; Max Temp (none) -> 125; Min Temp (none) -> -40
