File: Rocket/Boards/JPole_Antenna/JPole_Antenna.kicad_pcb (KiCad board)
At the start: 2 copper layers, 180 x 40 mm, 2 parts, among them J1 Conn_Coaxial, T1 NCS1-112+

Commit message: jpole needs review
Parts:
- J1, T1: moved to B.Cu
- moved T1 43.1 mm to (37.6, 69.3)
- moved J1 41.2 mm to (30.8, 70.7)
Routing:
- net /J_Pole_1: track 0.00 -> 340.0 mm, vias 0 -> 2
- net /RF_Port: track 185.0 -> 4.51 mm
- net GND: vias 4 -> 0
Other:
- board size 180 x 40 mm -> 246.6 x 39.7 mm
