File: Rocket/Boards/JPole_Antenna/JPole_Antenna.kicad_sch (KiCad schematic)
At the start: 2 parts, among them J1 Conn_Coaxial, T1 NCS1-112+

Commit message: jpole updates, ready for review
Parts:
- J1: footprint Library:SMA-KE-16.5A_EdgeMount -> Library:SMA-KE-16.5A_EdgeMount (1)
Changed lines of the file:
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@@
 			)
 		)
-		(property "Footprint" "Library:SMA-KE-16.5A_EdgeMount"
+		(property "Footprint" "Library:SMA-KE-16.5A_EdgeMount (1)"
 			(at 184.15 74.93 0)
 			(hide yes)
