File: 03 Ground Station/Boards/GS_Radio/mircocontroller.kicad_sch (KiCad schematic)
At the start: 33 parts, among them J15 UART JST, J3 USB_B_Micro, J4 SWD JST PH, U4 STM32H562RGT6, Y2 12MHz

Commit message: rocket, gs, jpole need review b4 order, update last of bom
Parts:
- R2, R5: value R -> 0R; footprint (none) -> Resistor_SMD:R_0402_1005Metric
