File: 03 Ground Station/Boards/GS_Radio/power_connection.kicad_sch (KiCad schematic)
At the start: 14 parts, among them J11 MICROFIT, J5 MICROFIT, U5 MIC5365-3.3YC5, U6 MIC5365-3.3YC5, U7 AS78L05RTR-E1

Commit message: rocket, gs, jpole need review b4 order, update last of bom
Connections:
- net +7V4_In is gone; now on net +7V4_Input: J11.1 (Pin_1)
Changed lines of the file:
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@@
 		)
 	)
-	(label "+7V4_In"
+	(label "+V_In"
 		(at 26.67 125.73 0)
 		(effects
