File: 03 Ground Station/Boards/GS_Radio/rf_rocket_module.kicad_pcb (KiCad board)
At the start: 4 copper layers, 65 x 50 mm, 91 parts, among them J10 M80, J11 MICROFIT, J3 USB_B_Micro, J4 SWD JST PH, J5 MICROFIT, J6 RFIO SMA, J9 M80, U1 TCAN1046, U2 SX1262, U3 PE4259 RF Switch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

Commit message: rocket, gs, jpole need review b4 order, update last of bom
Parts:
- added J15: UART JST, Connector_JST:JST_PH_B3B-PH-K_1x03_P2.00mm_Vertical, F.Cu at (179.1, 103.0)
- added R2: 0R, Resistor_SMD:R_0402_1005Metric, F.Cu at (172.7, 106.3)
- added R5: 0R, Resistor_SMD:R_0402_1005Metric, F.Cu at (172.7, 105.3)
Connections:
- J11 pad 1: /Power Input/+7V4_In -> /Power Input/+V_In
- U4 pad 14: unconnected-(U4-PA0-Pad14) -> Net-(U4-PA0)
- U4 pad 15: unconnected-(U4-PA1-Pad15) -> Net-(U4-PA1)
Routing:
- net Net-(U4-PA1): track 0.00 -> 7.74 mm
- net Net-(U4-PA0): track 0.00 -> 7.52 mm
- net /MCU/UART_RX: track 0.00 -> 6.79 mm
- net /MCU/UART_TX: track 0.00 -> 6.14 mm
- net /Power Input/+7V4_In: track 5.71 -> 0.00 mm
- net /Power Input/+V_In: track 19.1 -> 24.8 mm
- net GND: track 76.3 -> 78.1 mm, vias 124 -> 125
Other:
- board text added: "UART"
