File: 02 Rocket/Boards/JPole_Antenna/JPole_Antenna.kicad_pcb (KiCad board)
At the start: 4 copper layers, 246.6 x 39.7 mm, 2 parts, among them J1 Conn_Coaxial, T1 NCS1-112+

Commit message: idk aye
Other:
- board size 246.6 x 39.7 mm -> 246.6 x 21.5 mm
Changed lines of the file:
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@@
 		(capping no)
 		(filling no)
-		(zone_defaults)
 		(pcbplotparams
 			(layerselection 0x00000000_00000000_55555555_5755f5ff)
@@
 	)
 	(gr_rect
-		(start 31 50.7)
-		(end 277.6 90.4)
+		(start 31 59.7)
+		(end 277.6 81.2)
 		(stroke
 			(width 0.2)

Commit message: Narottam Updates Resolved
Routing:
- net GND: vias 2 -> 3
Other:
- board text added: "J. Tomkins"
