File: 02 Rocket/Boards/JPole_Antenna/JPole_Antenna.kicad_pcb (KiCad board)
At the start: 4 copper layers, 246.6 x 21.5 mm, 2 parts, among them J1 Conn_Coaxial, T1 NCS1-112+

Commit message: updates to schematic notes
Routing:
- net /J_Pole_1: track 339.5 -> 361.9 mm
Other:
- board size 246.6 x 21.5 mm -> 267.9 x 21.5 mm
