File: 02 Rocket/Boards/Onboard_Radio/rf_rocket_module.kicad_sch (KiCad schematic)
At the start: 9 parts

Commit message: Narottam Updates Resolved
Parts:
- removed R20: 0R, Resistor_SMD:R_0603_1608Metric, symbol Device:R
Other:
- sheet CAN_Termination ports: added none; removed CAN_PWR_IN
- sheet LoRav2 ports: added none; removed +3V3A
- sheet MCU ports: added none; removed +3V3
- sheet Power Input ports: added none; removed +3V3A_Input, +3V3_Input, +5V_Input, +7V4_Input
