File: 02 Rocket/Boards/Onboard_Radio/power_connection.kicad_sch (KiCad schematic)
At the start: 14 parts, among them J11 MICROFIT, J5 MICROFIT, U5 MIC5365-3.3YC5, U6 MIC5365-3.3YC5, U7 AS78L05RTR-E1

Commit message: idk aye
Connections:
- net +V_In is gone; now on net +7V4_Input: C40.1, J5.1 (Pin_1), U7.3 (VIN)
Changed lines of the file:
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@@
 		)
 	)
-	(label "+7V4_In"
+	(label "+V_In"
 		(at 26.67 125.73 0)
 		(effects
@@
 		)
 	)
-	(label "+7V4_In"
+	(label "+V_In"
 		(at 208.28 116.84 0)
 		(effects

Commit message: Narottam Updates Resolved
Parts:
- added R10, R6: 10k, symbol Device:R
- U5, U6: value MIC5365-3.3YC5 -> SC573V33RTRC; LCSC Part # C73103 -> C3751903; MPN MIC5365-3.3YC5-TR -> SC573V33RTRC; Manufacturer MICROCHIP -> Semtech Corporation
- U7: value AS78L05RTR-E1 -> MC78M05BDTRKG; footprint Package_TO_SOT_SMD:SOT-89-3 -> Package_TO_SOT_SMD:TO-252-3_TabPin2; LCSC Part # C90471 -> (none); MPN AS78L05RTR-E1 -> MC78M05BDTRKG; Manufacturer DIODES -> onsemi
Connections:
- net +5V_LDO: now also R6.1
- net 3V3A_LDO_EN: now also R10.2
- net 3V3_LDO_EN: now also R6.2
- net GND: now also R10.1
- net +3V3A_Input renamed +3V3A
- net +3V3_Input renamed +3V3
- net +5V_Input renamed +5V
- net +7V4_Input renamed +V_In
Other:
- note added: "5V5 In Max, 3V3 Out"
- note added: "5V5 In Max, 3V3A Out"
- note added: "V_In, 5V Out"
- note removed: "5V In, 3V3 Out"
- note removed: "5V In, 3V3A Out"
- note removed: "7V4 In, 5V Out"
- moved on the sheet: C35, C36, C38, JP6, U5

Commit message: radio board ordered!
Parts:
- R10, R6: footprint (none) -> Resistor_SMD:R_0603_1608Metric; LCSC Part # (none) -> RC0603FR-0710KL; MPN (none) -> RC0603FR-0710KL; Manufacturer (none) -> YAGEO; Max Temp (none) -> 155; Min Temp (none) -> -55
Connections:
- net +V_In renamed +7V4
Changed lines of the file:
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@@
 	)
 	(junction
+		(at 100.33 165.1)
+		(diameter 0)
+		(color 0 0 0 0)
+	)
+	(junction
 		(at 105.41 43.18)
 		(diameter 0)
@@
 	(wire
 		(pts
-			(xy 102.87 165.1) (xy 92.71 165.1)
+			(xy 102.87 165.1) (xy 100.33 165.1)
 		)
 		(stroke
@@
 	(wire
 		(pts
+			(xy 100.33 165.1) (xy 92.71 165.1)
+		)
+		(stroke
+			(width 0)
+			(type default)
+		)
+	)
+	(wire
+		(pts
 			(xy 105.41 43.18) (xy 121.92 43.18)
 		)
@@
 			)
 		)
-		(property "Footprint" ""
+		(property "Footprint" "Resistor_SMD:R_0603_1608Metric"
 			(at 121.92 113.538 90)
 			(hide yes)
@@
 			)
 		)
-		(property "Datasheet" ""
+		(property "Datasheet" "https://yageogroup.com/content/datasheet/asset/file/PYU-RC_GROUP_51_ROHS_L"
 			(at 121.92 111.76 0)
 			(hide yes)
@@
 			)
 		)
-		(property "Description" "Resistor"
+		(property "Description" "10 kOhms ±1% 0.1W, 1/10W Chip Resistor 0603 (1608 Metric) Moisture Resistant Thick Film"
 			(at 121.92 111.76 0)
 			(hide yes)
@@
 			)
 		)
+		(property "LCSC Part #" "RC0603FR-0710KL"
+			(at 121.92 111.76 90)
+			(hide yes)
+			(show_name no)
+			(do_not_autoplace no)
+			(effects
+				(font
+					(size 1.27 1.27)
+				)
+			)
+		)
+		(property "MPN" "RC0603FR-0710KL"
+			(at 121.92 111.76 90)
+			(hide yes)
+			(show_name no)
+			(do_not_autoplace no)
+			(effects
+				(font
+					(size 1.27 1.27)
+				)
+			)
+		)
+		(property "Manufacturer" "YAGEO"
+			(at 121.92 111.76 90)
+			(hide yes)
+			(show_name no)
+			(do_not_autoplace no)
+			(effects
+				(font
+					(size 1.27 1.27)
+				)
+			)
+		)
+		(property "Max Temp" "155"
+			(at 121.92 111.76 90)
+			(hide yes)
+			(show_name no)
+			(do_not_autoplace no)
+			(effects
+				(font
+					(size 1.27 1.27)
+				)
+			)
+		)
+		(property "Min Temp" "-55"
+			(at 121.92 111.76 90)
+			(hide yes)
+			(show_name no)
+			(do_not_autoplace no)
+			(effects
+				(font
+					(size 1.27 1.27)
+				)
+			)
+		)
 		(pin "1"
 		)
@@
 			)
 		)
-		(property "Footprint" ""
+		(property "Footprint" "Resistor_SMD:R_0603_1608Metric"
 			(at 113.03 50.038 90)
 			(hide yes)
@@
 			)
 		)
-		(property "Datasheet" ""
+		(property "Datasheet" "https://yageogroup.com/content/datasheet/asset/file/PYU-RC_GROUP_51_ROHS_L"
 			(at 113.03 48.26 0)
 			(hide yes)
@@
 			)
 		)
-		(property "Description" "Resistor"
+		(property "Description" "10 kOhms ±1% 0.1W, 1/10W Chip Resistor 0603 (1608 Metric) Moisture Resistant Thick Film"
 			(at 113.03 48.26 0)
 			(hide yes)
@@
 			)
 		)
+		(property "LCSC Part #" "RC0603FR-0710KL"
+			(at 113.03 48.26 90)
+			(hide yes)
+			(show_name no)
+			(do_not_autoplace no)
+			(effects
+				(font
+					(size 1.27 1.27)
+				)
+			)
+		)
+		(property "MPN" "RC0603FR-0710KL"
+			(at 113.03 48.26 90)
+			(hide yes)
+			(show_name no)
+			(do_not_autoplace no)
+			(effects
+				(font
+					(size 1.27 1.27)
+				)
+			)
+		)
+		(property "Manufacturer" "YAGEO"
+			(at 113.03 48.26 90)
+			(hide yes)
+			(show_name no)
+			(do_not_autoplace no)
+			(effects
+				(font
+					(size 1.27 1.27)
+				)
+			)
+		)
+		(property "Max Temp" "155"
+			(at 113.03 48.26 90)
+			(hide yes)
+			(show_name no)
+			(do_not_autoplace no)
+			(effects
+				(font
+					(size 1.27 1.27)
+				)
+			)
+		)
+		(property "Min Temp" "-55"
+			(at 113.03 48.26 90)
+			(hide yes)
+			(show_name no)
+			(do_not_autoplace no)
+			(effects
+				(font
+					(size 1.27 1.27)
+				)
+			)
+		)
 		(pin "2"
 		)
@@
 					(unit 1)
 				)
+			)
+		)
+	)
+	(symbol
+		(lib_id "power:+7.5V")
+		(at 100.33 165.1 0)
+		(unit 1)
+		(body_style 1)
+		(exclude_from_sim no)
+		(in_bom yes)
+		(on_board yes)
+		(in_pos_files yes)
+		(dnp no)
+		(fields_autoplaced yes)
+		(property "Reference" "#PWR056"
+			(at 100.33 168.91 0)
+			(hide yes)
+			(show_name no)
+			(do_not_autoplace no)
+			(effects
+				(font
+					(size 1.27 1.27)
+				)
+			)
+		)
+		(property "Value" "+7V4"
+			(at 100.33 160.02 0)
+			(show_name no)
+			(do_not_autoplace no)
+			(effects
+				(font
+					(size 1.27 1.27)
+				)
+			)
+		)
+		(property "Footprint" ""
+			(at 100.33 165.1 0)
+			(hide yes)
+			(show_name no)
+			(do_not_autoplace no)
+			(effects
+				(font
+					(size 1.27 1.27)
+				)
+			)
+		)
+		(property "Datasheet" ""
+			(at 100.33 165.1 0)
+			(hide yes)
+			(show_name no)
+			(do_not_autoplace no)
+			(effects
+				(font
+					(size 1.27 1.27)
+				)
+			)
+		)
+		(property "Description" "Power symbol creates a global label with name \"+7.5V\""
+			(at 100.33 165.1 0)
+			(hide yes)
+			(show_name no)
+			(do_not_autoplace no)
+			(effects
+				(font
+					(size 1.27 1.27)
+				)
+			)
+		)
+		(pin "1"
+		)
+		(instances
+			(project "rf_rocket_module"
+				(path "/4940ffbe-f45f-4917-a247-12e2b32b6c35/abcae1e2-b29e-4289-bda9-47e90da98056"
+					(reference "#PWR056")
+					(unit 1)
+				)
